Commit message: Eth_quad_with_payload

File: rotors_description/urdf/iris.xacro (robot description, xacro)
@@ -130,3 +130,27 @@
     <xacro:insert_block name="rotor_inertia" />
   </xacro:vertical_rotor>
+  <xacro:property name="arm_length" value="0.6" />
+  <xacro:property name="mass_arm" value="0.01" />
+  <link name="box">
+    <xacro:box_inertial x="${arm_length}" y="0.03" z="0.01" mass="0.01">
+      <origin xyz="${arm_length/2} 0 0" />
+    </xacro:box_inertial>
+    <visual>
+      <origin xyz="${arm_length/2} 0 0" rpy="0 0 0" />
+      <geometry>
+        <box size="0.2 0.2 0.2"/> <!-- [m] [m] [m] -->
+      </geometry>
+    </visual>
+    <collision>
+      <origin xyz="${arm_length/2} 0 0" rpy="0 0 0" />
+      <geometry>
+        <box size="$0.2 0.2 0.2"/> <!-- [m] [m] [m] -->
+      </geometry>
+    </collision>
+  </link>
+    <joint name="${namespace}/base_joint_box" type="fixed">
+      <origin xyz="-0.3 0 -0.12" rpy="0 0 0" />
+      <parent link="${namespace}/base_link" />
+      <child link="box" />
+    </joint>
 </robot>

Commit message: Box

File: rotors_description/urdf/iris.xacro (robot description, xacro)
@@ -132,6 +132,6 @@
   <xacro:property name="arm_length" value="0.6" />
   <xacro:property name="mass_arm" value="0.01" />
-  <link name="box">
-    <xacro:box_inertial x="${arm_length}" y="0.03" z="0.01" mass="0.01">
+   <link name="box">
+    <xacro:box_inertial x="${arm_length}" y="0.03" z="0.01" mass="0.3">
       <origin xyz="${arm_length/2} 0 0" />
     </xacro:box_inertial>
@@ -146,5 +146,5 @@
       <geometry>
         <box size="$0.2 0.2 0.2"/> <!-- [m] [m] [m] -->
-      </geometry>
+       </geometry>
     </collision>
   </link>

Commit message: PD controller

File: rotors_description/urdf/iris.xacro (robot description, xacro)
@@ -16,9 +16,10 @@
   <xacro:property name="rotor_offset_top" value="0.023" /> <!-- [m] -->
   <xacro:property name="radius_rotor" value="0.1" /> <!-- [m] -->
-  <xacro:property name="motor_constant" value="8.54858e-06" /> <!-- [kg.m/s^2] -->
+  <xacro:property name="motor_constant" value="12.44460e-06" /> <!-- [kg.m/s^2] -->
+  <!-- for default = 8.54858e-06  --> <!-- for 0.3 kg = 10.44460e-06  -->
   <xacro:property name="moment_constant" value="0.016" /> <!-- [m] -->
   <xacro:property name="time_constant_up" value="0.0125" /> <!-- [s] -->
   <xacro:property name="time_constant_down" value="0.025" /> <!-- [s] -->
-  <xacro:property name="max_rot_velocity" value="838" /> <!-- [rad/s] -->
+  <xacro:property name="max_rot_velocity" value="1200" /> <!-- [rad/s] -->
   <xacro:property name="sin30" value="0.5" />
   <xacro:property name="cos30" value="0.866025403784" />
@@ -30,4 +31,8 @@
     <inertia ixx="0.0347563" ixy="0.0" ixz="0.0" iyy="0.0458929" iyz="0.0" izz="0.0977" /> <!-- [kg.m^2] [kg.m^2] [kg.m^2] [kg.m^2] [kg.m^2] [kg.m^2] -->
   </xacro:property>
+<!--      MODIFIED INERTIA  FOR m = 0.3       -->
+  <!-- <xacro:property name="body_inertia">
+    <inertia ixx="0.0397563" ixy="0.0" ixz="0.0" iyy="0.0508929" iyz="0.0" izz="0.1077" />
+   </xacro:property> -->
   <!-- inertia of a single rotor, assuming it is a cuboid. Height=3mm, width=15mm -->
   <xacro:property name="rotor_inertia">
@@ -133,5 +138,5 @@
   <xacro:property name="mass_arm" value="0.01" />
    <link name="box">
-    <xacro:box_inertial x="${arm_length}" y="0.03" z="0.01" mass="0.3">
+    <xacro:box_inertial x="${arm_length}" y="0.03" z="0.01" mass="1">
       <origin xyz="${arm_length/2} 0 0" />
     </xacro:box_inertial>

Commit message: rotors_pid

File: rotors_description/urdf/iris.xacro (robot description, xacro)
@@ -133,9 +133,9 @@
   <xacro:property name="mass_arm" value="0.01" />
    <link name="box">
-    <xacro:box_inertial x="${arm_length}" y="0.03" z="0.01" mass="0.3">
-      <origin xyz="${arm_length/2} 0 0" />
+    <xacro:box_inertial x="-0.1" y="-0.1" z="-0.1" mass="0.3">
+      <origin xyz="0 0 0" />
     </xacro:box_inertial>
     <visual>
-      <origin xyz="${arm_length/2} 0 0" rpy="0 0 0" />
+      <origin xyz="0 0 0" rpy="0 0 0" />
       <geometry>
         <box size="0.2 0.2 0.2"/> <!-- [m] [m] [m] -->
@@ -143,12 +143,12 @@
     </visual>
     <collision>
-      <origin xyz="${arm_length/2} 0 0" rpy="0 0 0" />
+      <origin xyz="0 0 0" rpy="0 0 0" />
       <geometry>
-        <box size="$0.2 0.2 0.2"/> <!-- [m] [m] [m] -->
+        <box size="0.2 0.2 0.2"/> <!-- [m] [m] [m] -->
        </geometry>
     </collision>
   </link>
     <joint name="${namespace}/base_joint_box" type="fixed">
-      <origin xyz="-0.3 0 -0.12" rpy="0 0 0" />
+      <origin xyz="0 0 -0.12" rpy="0 0 0" />
       <parent link="${namespace}/base_link" />
       <child link="box" />

Commit message: Lidar added

File: rotors_description/urdf/iris.xacro (robot description, xacro)
@@ -130,8 +130,6 @@
     <xacro:insert_block name="rotor_inertia" />
   </xacro:vertical_rotor>
-  <xacro:property name="arm_length" value="0.6" />
-  <xacro:property name="mass_arm" value="0.01" />
-   <link name="box">
-    <xacro:box_inertial x="-0.1" y="-0.1" z="-0.1" mass="0.3">
+     <link name="box">
+    <xacro:box_inertial x="-0.1" y="-0.1" z="-0.1" mass="0.8">
       <origin xyz="0 0 0" />
     </xacro:box_inertial>
@@ -139,5 +137,5 @@
       <origin xyz="0 0 0" rpy="0 0 0" />
       <geometry>
-        <box size="0.2 0.2 0.2"/> <!-- [m] [m] [m] -->
+        <box size="0.2 0.2 0.2"/>
       </geometry>
     </visual>
@@ -145,5 +143,5 @@
       <origin xyz="0 0 0" rpy="0 0 0" />
       <geometry>
-        <box size="0.2 0.2 0.2"/> <!-- [m] [m] [m] -->
+        <box size="0.2 0.2 0.2"/>
        </geometry>
     </collision>
@@ -154,3 +152,7 @@
       <child link="box" />
     </joint>
+ <xacro:hokuyo_utm30lx robot_namespace="${namespace}" min_angle="-1.047" max_angle="1.047"
+    update_rate="40" ray_count="10">
+    <origin xyz="0 0 0.5" rpy="0 0 0"/>
+  </xacro:hokuyo_utm30lx>
 </robot>

File: rotors_description/urdf/multirotor_base.xacro (robot description, xacro)
@@ -132,3 +132,63 @@
     </gazebo>
   </xacro:macro>
+ <!-- Hokuyo Lidar Range Sensor -->
+    <xacro:macro name="hokuyo_utm30lx" params="robot_namespace *origin update_rate ray_count min_angle max_angle">
+      <link name="${robot_namespace}/laser_lidar_link12">
+  <inertial>
+    <mass value="0.001" />
+    <origin xyz="0 0 0" rpy="0 0 0" />
+    <inertia ixx="0.0001" ixy="0" ixz="0" iyy="0.0001" iyz="0" izz="0.0001" />
+  </inertial>
+  <visual>
+          <geometry>
+            <!--<mesh filename="package://turtlebot_description/meshes/sensors/hokuyo_utm30lx/hokuyo_utm_30lx.dae"/> -->
+            <box size="0.05 0.05 0.02"/>
+          </geometry>
+  </visual>
+  <collision>
+    <origin xyz="0 0 -0.0115" rpy="0 0 0" />
+          <geometry>
+            <box size="0.058 0.058 0.087" />
+            <!--<mesh filename="package://hector_sensors_description/meshes/hokuyo_utm30lx/hokuyo_utm_30lx.stl"/>-->
+          </geometry>
+  </collision>
+      </link>
+      <joint name="laser_lidar_joint" type="fixed">
+        <origin xyz="0.0 0.0 0.12" rpy="3.14159 0.0 0.0" />
+  <parent link="${robot_namespace}/base_link"/>
+  <child link="${robot_namespace}/laser_lidar_link12"/>
+      </joint>
+      <gazebo reference="${robot_namespace}/laser_lidar_link12">
+        <sensor type="ray" name="iris_laser_lidar">
+            <pose>0 0 0 0 0 0</pose>
+            <visualize>false</visualize>
+            <update_rate>1</update_rate>
+      <ray>
+      <scan>
+        <horizontal>
+          <samples>3</samples>
+          <resolution>10</resolution>
+          <min_angle>-1</min_angle>
+          <max_angle>1</max_angle>
+        </horizontal>
+      </scan>
+      <range>
+        <min>0.10</min>
+        <max>20.0</max>
+        <resolution>0.01</resolution>
+      </range>
+      <noise>
+        <type>Gaussian</type>
+        <mean>0.0</mean>
+        <stddev>0.01</stddev>
+      </noise>
+      </ray>
+      <plugin name="ray" filename="libgazebo_ros_laser.so">
+      <topicName>/scan</topicName>
+      <frameName>iris/laser_lidar_link12</frameName>
+      <!-- <interface:laser name="gazebo_ros_${laser_suffix}_iface" /> -->
+            </plugin>
+        </sensor>
+      </gazebo>
+    </xacro:macro>
 </robot>

Commit message: octomap_server added

File: rotors_description/urdf/iris.xacro (robot description, xacro)
@@ -20,5 +20,5 @@
   <xacro:property name="time_constant_up" value="0.0125" /> <!-- [s] -->
   <xacro:property name="time_constant_down" value="0.025" /> <!-- [s] -->
-  <xacro:property name="max_rot_velocity" value="838" /> <!-- [rad/s] -->
+  <xacro:property name="max_rot_velocity" value="2000" /> <!-- [rad/s] -->
   <xacro:property name="sin30" value="0.5" />
   <xacro:property name="cos30" value="0.866025403784" />
@@ -131,5 +131,5 @@
   </xacro:vertical_rotor>
      <link name="box">
-    <xacro:box_inertial x="-0.1" y="-0.1" z="-0.1" mass="0.8">
+    <xacro:box_inertial x="-0.1" y="-0.1" z="-0.1" mass="0.1">
       <origin xyz="0 0 0" />
     </xacro:box_inertial>
@@ -152,7 +152,6 @@
       <child link="box" />
     </joint>
- <xacro:hokuyo_utm30lx robot_namespace="${namespace}" min_angle="-1.047" max_angle="1.047"
-    update_rate="40" ray_count="10">
-    <origin xyz="0 0 0.5" rpy="0 0 0"/>
-  </xacro:hokuyo_utm30lx>
+<xacro:velodyne name="lidar" parent="${namespace}/base_link">
+  <origin xyz="0.0 0.0 0.1" rpy="0 0 0"/>
+</xacro:velodyne>
 </robot>

File: rotors_description/urdf/multirotor_base.xacro (robot description, xacro)
@@ -132,63 +132,89 @@
     </gazebo>
   </xacro:macro>
- <!-- Hokuyo Lidar Range Sensor -->
-    <xacro:macro name="hokuyo_utm30lx" params="robot_namespace *origin update_rate ray_count min_angle max_angle">
-      <link name="${robot_namespace}/laser_lidar_link12">
-  <inertial>
-    <mass value="0.001" />
-    <origin xyz="0 0 0" rpy="0 0 0" />
-    <inertia ixx="0.0001" ixy="0" ixz="0" iyy="0.0001" iyz="0" izz="0.0001" />
-  </inertial>
-  <visual>
-          <geometry>
-            <!--<mesh filename="package://turtlebot_description/meshes/sensors/hokuyo_utm30lx/hokuyo_utm_30lx.dae"/> -->
-            <box size="0.05 0.05 0.02"/>
-          </geometry>
-  </visual>
-  <collision>
-    <origin xyz="0 0 -0.0115" rpy="0 0 0" />
-          <geometry>
-            <box size="0.058 0.058 0.087" />
-            <!--<mesh filename="package://hector_sensors_description/meshes/hokuyo_utm30lx/hokuyo_utm_30lx.stl"/>-->
-          </geometry>
-  </collision>
-      </link>
-      <joint name="laser_lidar_joint" type="fixed">
-        <origin xyz="0.0 0.0 0.12" rpy="3.14159 0.0 0.0" />
-  <parent link="${robot_namespace}/base_link"/>
-  <child link="${robot_namespace}/laser_lidar_link12"/>
-      </joint>
-      <gazebo reference="${robot_namespace}/laser_lidar_link12">
-        <sensor type="ray" name="iris_laser_lidar">
-            <pose>0 0 0 0 0 0</pose>
-            <visualize>false</visualize>
-            <update_rate>1</update_rate>
-      <ray>
-      <scan>
-        <horizontal>
-          <samples>3</samples>
-          <resolution>10</resolution>
-          <min_angle>-1</min_angle>
-          <max_angle>1</max_angle>
-        </horizontal>
-      </scan>
-      <range>
-        <min>0.10</min>
-        <max>20.0</max>
-        <resolution>0.01</resolution>
-      </range>
-      <noise>
-        <type>Gaussian</type>
-        <mean>0.0</mean>
-        <stddev>0.01</stddev>
-      </noise>
-      </ray>
-      <plugin name="ray" filename="libgazebo_ros_laser.so">
-      <topicName>/scan</topicName>
-      <frameName>iris/laser_lidar_link12</frameName>
-      <!-- <interface:laser name="gazebo_ros_${laser_suffix}_iface" /> -->
-            </plugin>
-        </sensor>
-      </gazebo>
-    </xacro:macro>
+  <!-- Velodyne Lidar -->
+  <xacro:macro name="velodyne_sensor" params="link_name frame_name lidar_name">
+    <gazebo reference="${link_name}">
+      <sensor name="${link_name}_velodyne_sensor" type="ray">
+        <always_on>true</always_on>
+        <visualize>true</visualize>
+        <update_rate>1.0</update_rate>
+        <pose>0 0 0 0 0 0</pose>
+        <ray>
+          <scan>
+            <horizontal>
+              <samples>360</samples>
+              <resolution>1</resolution>
+              <min_angle>-3.14</min_angle>
+              <max_angle>3.14</max_angle>
+            </horizontal>
+            <vertical>
+              <samples>30</samples>
+              <resolution>1</resolution>
+              <min_angle>-20</min_angle>
+              <max_angle>10</max_angle>
+            </vertical>
+          </scan>
+          <range>
+            <min>0,3</min>
+            <max>5.0</max>
+            <resolution>0.02</resolution>
+          </range>
+        </ray>
+        <!-- test plugin -->
+        <plugin name="${link_name}_controller" filename="libgazebo_ros_laser.so">
+          <gaussianNoise>0.005</gaussianNoise>
+          <alwaysOn>true</alwaysOn>
+          <updateRate>10</updateRate>
+          <topicName>/scan</topicName>
+          <frameName>${frame_name}</frameName>
+          <hokuyoMinIntensity>101</hokuyoMinIntensity>
+        </plugin>
+      </sensor>
+    </gazebo>
+  </xacro:macro>
+  <xacro:macro name="velodyne" params="name parent *origin">
+    <!-- Joints -->
+    <joint name="${name}_joint" type="fixed">
+      <xacro:insert_block name="origin"/>
+      <parent link="${parent}"/>
+      <child link="${name}_mount_link"/>
+    </joint>
+    <!-- velodyne sensor optical frame -->
+    <joint name="${name}_optical_frame_joint" type="fixed">
+      <origin xyz="0.0 0.0 0.02" rpy="0.0 0.0 0.0"/>
+      <parent link="${name}_mount_link"/>
+      <child link="${name}"/>
+    </joint>
+    <!-- Velodyne Links -->
+    <link name="${name}_mount_link">
+      <xacro:box_inertial x="-0.02" y="-0.02" z="-0.01" mass="0.01">
+      <origin xyz="0 0 0" />
+    </xacro:box_inertial>
+      <visual>
+        <origin xyz="0 0 0" rpy="0 0 0"/>
+        <geometry>
+          <box size="0.05 0.05 0.02"/>
+        </geometry>
+        <material name="gray">
+          <color rgba="0.5 0.5 0.5 1"/>
+        </material>
+      </visual>
+      <collision>
+        <origin xyz="0 0 0" rpy="0 0 0"/>
+        <geometry>
+          <box size="0.05 0.05 0.02"/>
+        </geometry>
+      </collision>
+    </link>
+    <!-- rgb optical sensor link -->
+    <link name="${name}">
+      <inertial>
+        <mass value="0.1"/>
+        <origin xyz="0 0 0" rpy="0 0 0"/>
+        <inertia ixx="0.01" ixy="0.0" ixz="0.0" iyy="0.01" iyz="0.0" izz="0.01"/>
+      </inertial>
+    </link>
+    <!-- gazebo extensions -->
+    <xacro:velodyne_sensor link_name="${name}" frame_name="${name}_mount_link" lidar_name="${name}" />
+  </xacro:macro>
 </robot>

Commit message: read me

File: rotors_description/urdf/iris.xacro (robot description, xacro)
@@ -135,4 +135,216 @@
     <xacro:insert_block name="rotor_inertia" />
   </xacro:vertical_rotor>
+<!-- Mount a VI-sensor in the front of Neo.
+  <xacro:vi_sensor_macro
+      namespace="${namespace}/vi_sensor"
+      parent_link="${namespace}/base_link"
+      enable_cameras="true"
+      enable_depth="true"
+      enable_ground_truth="true">
+    <origin xyz="0.133 0.0 -0.0565" rpy="0.0 ${20.0/180.0*pi} 0.0" />
+  </xacro:vi_sensor_macro>
+  <xacro:vi_sensor_camera_macro
+      namespace="${namespace}/vi_sensor"
+      parent_link="${namespace}/base_link"
+      camera_suffix="2"
+      frame_rate="20">
+    <origin xyz="0.019 0.0 0.073" rpy="0.0 ${-pi/2} 0.0" />
+  </xacro:vi_sensor_camera_macro>
+  <xacro:vi_sensor_camera_macro
+      namespace="${namespace}/vi_sensor"
+      parent_link="${namespace}/base_link"
+      camera_suffix="3"
+      frame_rate="20">
+    <origin xyz="0.019 0.0 -0.045" rpy="0.0 ${pi/2} 0.0" />
+  </xacro:vi_sensor_camera_macro>     -->
+<!--
+  <gazebo reference="sensor">
+    <sensor type="ray" name="head_hokuyo_sensor">
+      <pose>0 0 0 0 0 0</pose>
+      <visualize>false</visualize>
+      <update_rate>40</update_rate>
+      <ray>
+        <scan>
+          <horizontal>
+            <samples>720</samples>
+            <resolution>1</resolution>
+            <min_angle>-1.570796</min_angle>
+            <max_angle>1.570796</max_angle>
+          </horizontal>
+        </scan>
+        <range>
+          <min>0.8</min>
+          <max>30.0</max>
+          <resolution>0.01</resolution>
+        </range>
+        <noise>
+          <type>gaussian</type>
+          <mean>0.0</mean>
+          <stddev>0.01</stddev>
+        </noise>
+      </ray>
+      <plugin name="gazebo_ros_head_hokuyo_controller" filename="libgazebo_ros_laser.so">
+        <topicName>/laser/scan</topicName>
+        <frameName>world</frameName>
+      </plugin>
+    </sensor>
+</gazebo> -->
+<!-- <link name="laser">
+    <inertial>
+      <xacro:hokuyo_inertial_params />
+    </inertial>
+    <origin xyz="0 0 0" rpy="0 0 0" />
+  <mass value="0.100" />
+  <inertia ixx="4E-06" ixy="0"           ixz="0"
+                            iyy="4E-06"  iyz="0"
+                                         izz="4E-06" />
+    <collision>
+      <origin xyz="0 0 0" rpy="0 0 0"/>
+      <geometry>
+        <box size="0.1 0.1 0.1"/>
+      </geometry>
+    </collision>
+    <visual>
+      <origin xyz="0 0 0" rpy="0 0 0"/>
+      <geometry>
+        <box size = "0.1 0.1 0.1"/>
+      </geometry>
+    </visual>
+  </link>
+  <joint name="hokuyo_joint" type="fixed">
+    <origin xyz="2 0 2" rpy="0 0 0"/>
+    <parent link="${namespace}/base_link" />
+    <child link="laser" />
+    <axis xyz="0 0 1" />
+</joint>
+-->
+<!--
+<xacro:macro name="hokuyo_laser" params="xyz rpy parent">
+    <joint name="hokuyo_laser_joint" type="fixed">
+        <axis xyz="0 0 1" />
+        <origin xyz="${xyz}" rpy="${rpy}"/>
+        <parent link="${namespace}/base_link"/>
+        <child link="hokuyo_laser_link"/>
+    </joint>
+    <link name="hokuyo_laser_link">
+        <collision>
+            <origin xyz="0 0 0" rpy="0 0 0"/>
+            <geometry>
+                <cylinder length="0.04" radius="0.045"/>
+            </geometry>
+        </collision>
+        <visual>
+            <origin xyz="0 0 0" rpy="0 0 0"/>
+            <geometry>
+                <cylinder length="0.04" radius="0.045"/>
+            </geometry>
+        </visual>
+        <inertial>
+            <mass value="1e-5" />
+            <origin xyz="0 0 0" rpy="0 0 0"/>
+            <inertia ixx="1e-6" ixy="0" ixz="0" iyy="1e-6" iyz="0" izz="1e-6" />
+        </inertial>
+    </link>
+    <gazebo reference="hokuyo_laser_link">
+        <gravity>true</gravity>
+        <sensor type="ray" name="head_hokuyo_sensor">
+            <pose>0 0 0 0 0 0</pose>
+            <visualize>true</visualize>
+            <update_rate>40</update_rate>
+            <ray>
+                <scan>
+                    <horizontal>
+                        <samples>360</samples>
+                        <resolution>1</resolution>
+                        <min_angle>-3.14159</min_angle>
+                        <max_angle>3.14159</max_angle>
+                    </horizontal>
+                </scan>
+                <range>
+                    <min>0.2</min>
+                    <max>40</max>
+                    <resolution>0.025</resolution>
+                </range>
+                <noise>
+                    <type>gaussian</type>
+                    <mean>0.0</mean>
+                    <stddev>0.0</stddev>
+                </noise>
+            </ray>
+            <plugin name="gazebo_ros_head_hokuyo_controller" filename="libgazebo_ros_laser.so">
+                <robotNamespace></robotNamespace>
+                <topicName>laser_scan</topicName>
+                <frameName>hokuyo_laser_link</frameName>
+            </plugin>
+        </sensor>
+    </gazebo>
+</xacro:macro> -->
+<!-- <xacro:include filename="$(find hector_sensors_description)/urdf/hokuyo_utm30lx.urdf.xacro"/>
+<hokuyo_utm30lx_model name="hokuyo_laser" parent="base_link">
+  <origin xyz="0 0 +0.30" rpy="0 0 0" />
+</hokuyo_utm30lx_model> -->
+  <xacro:macro name="sick_lms1xx" params="frame:=laser topic:=scan sample_size:=720 update_rate:=50
+               min_angle:=-2.35619 max_angle:=2.35619 min_range:=0.1 max_range:=30.0 robot_namespace:=/" >
+    <link name="${frame}">
+      <inertial>
+        <mass value="1.1" />
+        <origin xyz="0 0 0" />
+        <inertia ixx="${0.0833333 * 1.1 * (0.102*0.102 + 0.152*0.152)}" ixy="0.0" ixz="0.0"
+          iyy="${0.0833333 * 1.1 * (0.105*0.105 + 0.152*0.152)}" iyz="0.0"
+          izz="${0.0833333 * 1.1 * (0.105*0.105 + 0.102*0.102)}" />
+      </inertial>
+      <visual>
+        <origin xyz="0 0 0" rpy="0 0 0" />
+        <geometry>
+          <!-- Origin of this mesh is the focal point of the LIDAR. -->
+          <mesh filename="package://lms1xx/meshes/sick-lms1xx.dae" />
+        </geometry>
+      </visual>
+      <collision>
+        <origin xyz="0 0 -0.05" rpy="0 0 0" />
+        <geometry>
+          <box size="0.105 0.1 0.1" />
+        </geometry>
+      </collision>
+    </link>
+    <joint name="${namespace}/base_joint_box" type="fixed">
+      <origin xyz="-0.3 0 -0.12" rpy="0 0 0" />
+      <parent link="${namespace}/base_link" />
+      <child link="${frame}" />
+    </joint>
+    <gazebo reference="${frame}">
+      <turnGravityOff>true</turnGravityOff>
+      <sensor type="ray" name="${frame}">
+        <pose>0 0 0 0 0 0</pose>
+        <visualize>false</visualize>
+        <update_rate>${update_rate}</update_rate>
+        <ray>
+          <scan>
+            <horizontal>
+              <samples>${sample_size}</samples>
+              <resolution>1</resolution>
+              <min_angle>${min_angle}</min_angle>
+              <max_angle>${max_angle}</max_angle>
+            </horizontal>
+          </scan>
+          <range>
+            <min>${min_range}</min>
+            <max>${max_range}</max>
+            <resolution>0.01</resolution>
+          </range>
+          <noise>
+            <type>gaussian</type>
+            <mean>0.0</mean>
+            <stddev>0.001</stddev>
+          </noise>
+        </ray>
+        <plugin name="gazebo_ros_laser" filename="libgazebo_ros_laser.so">
+          <topicName>${topic}</topicName>
+          <frameName>${frame}</frameName>
+          <robotNamespace>${robot_namespace}</robotNamespace>
+        </plugin>
+      </sensor>
+    </gazebo>
+</xacro:macro>
   <xacro:property name="arm_length" value="0.6" />
   <xacro:property name="mass_arm" value="0.01" />
@@ -150,5 +362,5 @@
       <origin xyz="${arm_length/2} 0 0" rpy="0 0 0" />
       <geometry>
-        <box size="$0.2 0.2 0.2"/> <!-- [m] [m] [m] -->
+        <box size="0.2 0.2 0.2"/> <!-- [m] [m] [m] -->
        </geometry>
     </collision>
